File: TSAL-board/TSAL-board.kicad_pcb (KiCad board)
At the start: 2 copper layers, 0 parts

Commit message: 完成、未チェック
チェック後、ガーバー出力
Parts:
- added C1: 0.1u, Capacitor_SMD:C_0603_1608Metric, F.Cu at (8.00, 37.5)
- added C10: 1000p, Capacitor_SMD:C_1206_3216Metric, F.Cu at (12.5, 3.00)
- added C2: 10u, Capacitor_SMD:C_1206_3216Metric, F.Cu at (9.00, 33.5)
- added C3: 10u, Capacitor_SMD:C_1206_3216Metric, F.Cu at (4.00, 33.5)
- added C4: 10u, Capacitor_SMD:C_1206_3216Metric, F.Cu at (9.00, 30.5)
- added C5: 10u, Capacitor_SMD:C_1206_3216Metric, F.Cu at (4.00, 30.5)
- added C6: 1u, Capacitor_SMD:C_0805_2012Metric, F.Cu at (15.5, 21.5)
- added C7: 1u, Capacitor_SMD:C_0805_2012Metric, F.Cu at (8.50, 26.0)
- added C8: 0.1u, Capacitor_SMD:C_0603_1608Metric, F.Cu at (8.50, 24.0)
- added C9: 10n, Capacitor_SMD:C_0603_1608Metric, F.Cu at (4.50, 16.5)
- added D1: PZ1AH11B-AU, ProjectEV:D_SOD-123HE_PZ1AHxxxB-AU, F.Cu at (14.5, 35.0)
- added D2: DFLZ24Q-7, ProjectEV:D_PowerDI-123_DFLZxxQ, F.Cu at (45.5, 7.50)
- added D3: DFLZ24Q-7, ProjectEV:D_PowerDI-123_DFLZxxQ, F.Cu at (54.5, 9.50)
- added D4: LED, LED_SMD:LED_0603_1608Metric, F.Cu at (4.00, 37.5)
- added F1: 0ABB-1000-TM, ProjectEV:Fuse_0ABB, F.Cu at (9.75, 40.5)
- added G***: Logo_TUT_10x10mm, ProjectEV:Logo_TUT_10x10mm, F.Cu at (23.0, 17.0)
- added G***: ISO_7010_W012, ProjectEV:ISO_7010_W012_10x8.7mm, F.Cu at (55.0, 55.0)
- added G***: ISO_7010_W012, ProjectEV:ISO_7010_W012_10x8.7mm, B.Cu at (55.0, 30.0)
- added H1: M3, MountingHole:MountingHole_3.2mm_M3_Pad_Via, F.Cu at (5.00, 5.00)
- added H2: M3, MountingHole:MountingHole_3.2mm_M3_Pad_Via, F.Cu at (77.5, 5.00)
- added H3: M3, MountingHole:MountingHole_3.2mm_M3_Pad_Via, F.Cu at (5.00, 60.0)
- added H4: M3, MountingHole:MountingHole_3.2mm_M3_Pad_Via, F.Cu at (77.5, 60.0)
- added J1: BM02B-PASS-1-TF, ProjectEV:Connector_BM02B-PASS-1-TF, F.Cu at (7.50, 47.5)
- added J2: 19427-0040, ProjectEV:Connector_MX150L_19427-0040, F.Cu at (73.9, 32.5)
- added J3: BM02B-PASS-1-TF, ProjectEV:Connector_BM02B-PASS-1-TF, F.Cu at (22.5, 40.0)
- added J4: BM02B-PASS-1-TF, ProjectEV:Connector_BM02B-PASS-1-TF, F.Cu at (22.5, 57.5)
- added Q1: DMP3098LQ-7, ProjectEV:Package_SOT-23_DMP3098LQ-7, F.Cu at (11.0, 37.5)
- added Q2: 2N7002K-AU, ProjectEV:Package_SOT-23_2N7002K-AU, F.Cu at (13.0, 12.5)
- added Q3: 2N7002K-AU, ProjectEV:Package_SOT-23_2N7002K-AU, F.Cu at (20.5, 31.5)
- added Q4: 2N7002K-AU, ProjectEV:Package_SOT-23_2N7002K-AU, F.Cu at (20.5, 49.5)
- added R1: 100k, Resistor_SMD:R_0603_1608Metric, F.Cu at (14.5, 39.5)
- added R10: 15.4k, Resistor_SMD:R_0603_1608Metric, F.Cu at (54.5, 6.00)
- added R11: 3.9k, Resistor_SMD:R_0603_1608Metric, F.Cu at (58.0, 6.00)
- added R12: 15k, ProjectEV:R_TEConnectivity_3502, F.Cu at (45.5, 55.5)
- added R13: 15k, ProjectEV:R_TEConnectivity_3502, F.Cu at (45.5, 45.5)
- added R14: 15k, ProjectEV:R_TEConnectivity_3502, F.Cu at (45.5, 35.5)
- added R15: 15k, ProjectEV:R_TEConnectivity_3502, F.Cu at (45.5, 25.5)
- added R16: 15k, ProjectEV:R_TEConnectivity_3502, F.Cu at (45.5, 15.5)
- added R17: 15k, ProjectEV:R_TEConnectivity_3502, F.Cu at (37.5, 55.5)
- added R18: 15k, ProjectEV:R_TEConnectivity_3502, F.Cu at (37.5, 45.5)
- added R19: 15k, ProjectEV:R_TEConnectivity_3502, F.Cu at (37.5, 35.5)
- added R2: 220k, ProjectEV:R_VishayDale_RCC1206-e3, F.Cu at (60.0, 42.0)
- added R20: 15k, ProjectEV:R_TEConnectivity_3502, F.Cu at (37.5, 25.5)
- added R21: 15k, ProjectEV:R_TEConnectivity_3502, F.Cu at (37.5, 15.5)
- added R22: 10k, Resistor_SMD:R_0603_1608Metric, F.Cu at (37.5, 9.00)
- added R23: 10k, Resistor_SMD:R_0603_1608Metric, F.Cu at (6.00, 37.5)
- added R24: 1M, Resistor_SMD:R_0603_1608Metric, F.Cu at (19.0, 27.5)
- added R25: 10k, Resistor_SMD:R_0603_1608Metric, F.Cu at (4.50, 23.5)
- added R26: 180k, Resistor_SMD:R_0603_1608Metric, F.Cu at (4.50, 20.0)
- added R27: 100, Resistor_SMD:R_0603_1608Metric, F.Cu at (16.5, 11.5)
- added R28: 100k, Resistor_SMD:R_0603_1608Metric, F.Cu at (12.2, 15.5)
- added R29: 1M, Resistor_SMD:R_1206_3216Metric, F.Cu at (12.5, 7.00)
- added R3: 220k, ProjectEV:R_VishayDale_RCC1206-e3, F.Cu at (60.0, 33.0)
- added R30: 100, Resistor_SMD:R_0603_1608Metric, F.Cu at (15.5, 47.5)
- added R31: 100, Resistor_SMD:R_0603_1608Metric, F.Cu at (21.0, 27.5)
- added R32: 1M, Resistor_SMD:R_0603_1608Metric, F.Cu at (17.5, 49.5)
- added R33: 0, Resistor_SMD:R_0603_1608Metric, F.Cu at (23.5, 31.5)
- added R34: 0, Resistor_SMD:R_0603_1608Metric, F.Cu at (23.5, 49.5)
- added R35: 100k, Resistor_SMD:R_0603_1608Metric, F.Cu at (14.5, 44.5)
- added R4: 220k, ProjectEV:R_VishayDale_RCC1206-e3, F.Cu at (60.0, 24.0)
- added R5: 220k, ProjectEV:R_VishayDale_RCC1206-e3, F.Cu at (60.0, 15.0)
- added R6: 220k, ProjectEV:R_VishayDale_RCC1206-e3, F.Cu at (53.0, 42.0)
- added R7: 220k, ProjectEV:R_VishayDale_RCC1206-e3, F.Cu at (53.0, 33.0)
- added R8: 220k, ProjectEV:R_VishayDale_RCC1206-e3, F.Cu at (53.0, 24.0)
- added R9: 220k, ProjectEV:R_VishayDale_RCC1206-e3, F.Cu at (53.0, 15.0)
- added REF**: Identifier_1pin, ProjectEV:Identifier_1pin, F.Cu at (38.5, 6.00)
- added REF**: Identifier_1pin, ProjectEV:Identifier_1pin, F.Cu at (12.8, 23.0)
- added REF**: Identifier_1pin, ProjectEV:Identifier_1pin, F.Cu at (23.5, 34.8)
- added REF**: Identifier_1pin, ProjectEV:Identifier_1pin, F.Cu at (8.50, 42.2)
- added REF**: Identifier_1pin, ProjectEV:Identifier_1pin, F.Cu at (23.5, 52.2)
- added REF**: Identifier_1pin, ProjectEV:Identifier_1pin, F.Cu at (65.5, 35.5)
- added REF**: Identifier_1pin, ProjectEV:Identifier_1pin, F.Cu at (35.0, 10.8)
- added U1: TL431QDBVR, ProjectEV:Package_SOT-23-5_TL431QDBVR, F.Cu at (41.0, 7.00)
- added U2: TLP291(GB,SE, ProjectEV:Isolator_TLP291(GB,SE, F.Cu at (32.0, 9.00)
- added U3: TLC555QDRQ1, ProjectEV:Package_SOIC-8_3.9x4.9mm_P1.27mm_TLC555QDRQ1, F.Cu at (10.0, 20.0)
Routing:
- net +12V: track 0.00 -> 82.6 mm, vias 0 -> 2
- net /TS-: track 0.00 -> 53.5 mm
- net /~{TS_ACTIVE}: track 0.00 -> 30.2 mm
- net /RED_SIG: track 0.00 -> 29.4 mm, vias 0 -> 2
- net Net-(D3-K): track 0.00 -> 20.2 mm, vias 0 -> 2
- net Net-(U3-THRES): track 0.00 -> 11.6 mm
- net Net-(D2-K): track 0.00 -> 9.35 mm
- net Net-(D1-A): track 0.00 -> 5.11 mm
- net Net-(U3-DISCH): track 0.00 -> 4.73 mm
- net Net-(U1-K): track 0.00 -> 4.72 mm
- net /~{RST}: track 0.00 -> 4.72 mm
- net Net-(J4-Pin_2): track 0.00 -> 4.70 mm
- net Net-(J3-Pin_2): track 0.00 -> 4.61 mm
- net /TSAL_GREEN_A: track 0.00 -> 4.38 mm
- net Net-(Q4-G): track 0.00 -> 4.20 mm
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- added copper zone on F.Cu, net +12V
- added copper zone on F.Cu, net /GLV_IN
- added copper zone on F.Cu, net /TS+
- added copper zone on B.Cu, net GND
- added copper zone on F.Cu, net GND
- added copper zone on B.Cu, net Net-(C10-Pad1)
- added copper zone on F.Cu, net Net-(C10-Pad1)
- added copper zone on F.Cu, net Net-(C2-Pad2)
- added copper zone on F.Cu, net Net-(C4-Pad2)
- added copper zone on F.Cu, net Net-(D2-K)
- added copper zone on F.Cu, net Net-(D3-K)
- added copper zone on F.Cu, net Net-(Q1-D)
- added copper zone on F.Cu, net Net-(R12-Pad2)
- added copper zone on F.Cu, net Net-(R13-Pad2)
- added copper zone on F.Cu, net Net-(R14-Pad2)
- added copper zone on F.Cu, net Net-(R15-Pad2)
- added copper zone on F.Cu, net Net-(R17-Pad2)
- added copper zone on F.Cu, net Net-(R18-Pad2)
- added copper zone on F.Cu, net Net-(R19-Pad2)
- added copper zone on F.Cu, net Net-(R2-Pad2)
- added copper zone on F.Cu, net Net-(R20-Pad2)
- added copper zone on F.Cu, net Net-(R3-Pad2)
- added copper zone on F.Cu, net Net-(R4-Pad2)
- added copper zone on F.Cu, net Net-(R6-Pad2)
- added copper zone on F.Cu, net Net-(R7-Pad2)
- added copper zone on F.Cu, net Net-(R8-Pad2)
Other:
- board outline added: 82.5 x 65 mm
- board text added: "4.00mm"
- board text added: "HIGH VOLTAGE"
- board text added: "POWER"
- board text added: "Project EV"
- board text added: "TSAL GREEN"
- board text added: "TSAL RED"
- board text added: "TSAL-board-v1.0"

Commit message: シルク修正
Parts:
- moved REF** 1.60 mm to (39.8, 5.00), turned to 0 degrees
Changed lines of the file:
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@@
   (net 47 "/TSAL_RED_A")
   (footprint "ProjectEV:Identifier_1pin" (layer "F.Cu")
-    (at 38.5 6 90)
+    (at 39.75 5)
     (attr allow_missing_courtyard)
-    (fp_text reference "REF**" (at 0 -0.5 90 unlocked) (layer "F.SilkS") hide
+    (fp_text reference "REF**" (at 0 -0.5 unlocked) (layer "F.SilkS") hide
         (effects (font (size 1 1) (thickness 0.1)))
     )
-    (fp_text value "Identifier_1pin" (at 0 1 90 unlocked) (layer "F.Fab")
-        (effects (font (size 1 1) (thickness 0.15)))
-    )
-    (fp_text user "▼" (at -0.375 0 90 unlocked) (layer "F.SilkS")
+    (fp_text value "Identifier_1pin" (at 0 1 unlocked) (layer "F.Fab")
+        (effects (font (size 1 1) (thickness 0.15)))
+    )
+    (fp_text user "▼" (at -0.375 0 unlocked) (layer "F.SilkS")
         (effects (font (size 0.8 0.5) (thickness 0.125) bold) (justify left bottom))
     )
-    (fp_text user "${REFERENCE}" (at 0 2.5 90 unlocked) (layer "F.Fab")
+    (fp_text user "${REFERENCE}" (at 0 2.5 unlocked) (layer "F.Fab")
         (effects (font (size 1 1) (thickness 0.15)))
     )
@@
     (property "ki_keywords" "R res resistor")
     (attr smd)
-    (fp_text reference "R22" (at 0 -1.5 90) (layer "F.SilkS")
-        (effects (font (size 1 1) (thickness 0.15)))
-    )
+    (fp_text reference "R22" (at 3 0 90) (layer "F.SilkS")
+        (effects (font (size 1 1) (thickness 0.15)))
+    )
